File: normie board.kicad_pcb (KiCad board)
At the start: 2 copper layers, 292.6 x 84.2 mm, 112 parts, among them SW1 SW_Push, U1 ATmega32U4-AU, U2 SRV05-4, Y1 16MHz

Commit message: NB46
Added a ground plane, and fixed all the disconnected traces, on paper it should work
Parts:
- moved C5 16.3 mm to (79.3, 113.7), turned to 90 degrees
Routing:
- net GND: track 14.6 -> 61.6 mm, vias 0 -> 12
- net +5V: track 129.1 -> 138.4 mm, vias 6 -> 7
- net GNDREF: track 21.6 -> 24.0 mm, vias 0 -> 1
- net Net-(R5-Pad2): track 10.1 -> 12.5 mm
- net DBUS-: track 18.3 -> 19.8 mm
- net ROW0: track 402.7 -> 404.0 mm
- net COL12: track 315.9 -> 317.0 mm
- net COL2: track 84.4 -> 85.5 mm
- net COL11: track 284.2 -> 285.4 mm
- added copper zone on B.Cu, net GND
- added copper zone on F.Cu, net GND
Other:
- board text added: "Designed by MelindaBirkenstock"

Commit message: rev whatever
Updated NB to have 19.05 spacing, and rearranged some trices
Parts:
- MX1, MX38, MX39, MX4, MX43: footprint Button_Switch_Keyboard:SW_Cherry_MX_1.50u_PCB -> Type-C:SW_Cherry_MX_1.00u_PCB_with_fixed_courtyard
- MX10, MX12, MX13, MX14, MX15, MX16, MX17, MX18, MX19, MX20, MX22, MX23, MX24, MX25, MX26, MX27, MX28, MX29, MX30, MX31, MX32, MX33, MX34, MX35, MX36, MX37, MX44, MX45, MX46, MX5, MX6, MX7, MX8, MX9: footprint Button_Switch_Keyboard:SW_Cherry_MX_1.00u_PCB -> Type-C:SW_Cherry_MX_1.00u_PCB_with_fixed_courtyard
- MX11, MX41: footprint Button_Switch_Keyboard:SW_Cherry_MX_1.25u_PCB -> Type-C:SW_Cherry_MX_1.00u_PCB_with_fixed_courtyard
- MX2, MX42: footprint Button_Switch_Keyboard:SW_Cherry_MX_1.75u_PCB -> Type-C:SW_Cherry_MX_1.00u_PCB_with_fixed_courtyard
- MX21, MX3: footprint Button_Switch_Keyboard:SW_Cherry_MX_2.25u_PCB -> Type-C:SW_Cherry_MX_2.25u_PCB_fixed_courtyard
- MX40: footprint Button_Switch_Keyboard:SW_Cherry_MX_2.75u_PCB -> Type-C:SW_Cherry_MX_2.75u_PCB_fixed_courtyard
- moved D45 7.00 mm to (296.0, 91.0)
- moved D44 6.75 mm to (291.0, 72.0)
- moved MX46 6.57 mm to (299.9, 76.0)
- moved MX44 6.56 mm to (295.2, 57.0)
- moved MX45 6.56 mm to (304.7, 95.1)
- moved D46 4.15 mm to (300.0, 109.0)
- moved MX31 2.49 mm to (157.1, 114.2)
- moved MX11 2.49 mm to (92.8, 114.2)
- moved MX21 2.49 mm to (126.2, 114.2)
- moved MX40 2.46 mm to (192.8, 114.2)
- moved D21 1.11 mm to (162.0, 109.0)
- moved D11 1.00 mm to (105.5, 109.0)
- moved D14 1.00 mm to (123.5, 109.0)
- moved D18 1.00 mm to (141.5, 109.0)
- moved D25 1.00 mm to (180.5, 109.0)
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Routing:
- net COL12: track 317.0 -> 300.6 mm
- net ROW0: track 404.0 -> 397.0 mm
- net ROW1: track 375.9 -> 369.0 mm
- net ROW2: track 360.8 -> 355.6 mm
- net COL1: track 82.1 -> 86.4 mm
- net Net-(D8-Pad2): track 18.6 -> 15.4 mm
- net COL3: track 116.0 -> 119.0 mm
- net Net-(D11-Pad2): track 20.1 -> 17.3 mm
- net COL6: track 187.4 -> 190.1 mm
- net Net-(D22-Pad2): track 19.0 -> 16.3 mm
- net COL2: track 85.5 -> 87.8 mm
- net COL5: track 147.0 -> 149.0 mm
- net Net-(D32-Pad2): track 18.3 -> 16.6 mm
- net Net-(D46-Pad2): track 13.2 -> 11.6 mm
- net COL7: track 186.2 -> 187.7 mm
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Other:
- board size 292.6 x 84.2 mm -> 285.9 x 84.7 mm
